File: pcb/testboard/motor_drive.kicad_sch (KiCad schematic)
At the start: 4 parts, among them IC1 TLE94112ESXUMA1, J3 52207-0633, J4 52207-0633, J5 52207-0633

Commit message: Final PCB Finished BOM and added MPN to all components
Parts:
- IC1: footprint (none) -> TLE94112ESXUMA1:SOP65P600X115-25N
- J3, J4, J5: Mouser Part Number (none) -> 52207-0633
Changed lines of the file:
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@@
 			)
 		)
-		(property "Datasheet" "http://www.molex.com/pdm_docs/sd/522072033_sd.pdf"
+		(property "Datasheet" "https://www.molex.com/en-us/products/part-detail/522072033"
 			(at 76.2 268.58 0)
 			(hide yes)
@@
 				)
 				(justify left top)
+			)
+		)
+		(property "Mouser Part Number" "52207-0633"
+			(at 59.69 73.66 0)
+			(hide yes)
+			(show_name no)
+			(do_not_autoplace no)
+			(effects
+				(font
+					(size 1.27 1.27)
+				)
 			)
 		)
@@
 			)
 		)
-		(property "Footprint" ""
+		(property "Footprint" "TLE94112ESXUMA1:SOP65P600X115-25N"
 			(at 173.99 176.2 0)
 			(hide yes)
@@
 			)
 		)
-		(property "Datasheet" "http://www.molex.com/pdm_docs/sd/522072033_sd.pdf"
+		(property "Datasheet" "https://www.molex.com/en-us/products/part-detail/522072033"
 			(at 76.2 286.36 0)
 			(hide yes)
@@
 				)
 				(justify left top)
+			)
+		)
+		(property "Mouser Part Number" "52207-0633"
+			(at 59.69 91.44 0)
+			(hide yes)
+			(show_name no)
+			(do_not_autoplace no)
+			(effects
+				(font
+					(size 1.27 1.27)
+				)
 			)
 		)
@@
 			)
 		)
-		(property "Datasheet" "http://www.molex.com/pdm_docs/sd/522072033_sd.pdf"
+		(property "Datasheet" "https://www.molex.com/en-us/products/part-detail/522072033"
 			(at 76.2 250.8 0)
 			(hide yes)
@@
 			)
 		)
+		(property "Mouser Part Number" "52207-0633"
+			(at 59.69 55.88 0)
+			(hide yes)
+			(show_name no)
+			(do_not_autoplace no)
+			(effects
+				(font
+					(size 1.27 1.27)
+				)
+			)
+		)
