File: pcb/testboard/testboard.kicad_sch (KiCad schematic)
At the start: 4 parts, among them J1 Left Socket, J2 Right Socket, SW1 Control

Commit message: Final PCB Finished BOM and added MPN to all components
Parts:
- J1, J2: Manufacturer_Part_Number (none) -> M20-7822046; Mouser Part Number (none) -> M20-7822046
- R5: Manufacturer_Part_Number (none) -> RC0805FR-071KL; Mouser Part Number (none) -> RC0805FR-071KL
- SW1: Manufacturer_Part_Number (none) -> B3F-4000; Mouser Part Number (none) -> B3F-4000
Changed lines of the file:
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@@
 			)
 		)
-		(property "Datasheet" ""
+		(property "Datasheet" "https://mm.digikey.com/Volume0/opasdata/d220001/medias/docus/937/Female_Headers.100_DS.pdf"
 			(at 123.19 76.2 0)
 			(hide yes)
@@
 		)
 		(property "Description" "Generic connector, single row, 01x20, script generated"
+			(at 123.19 76.2 0)
+			(hide yes)
+			(show_name no)
+			(do_not_autoplace no)
+			(effects
+				(font
+					(size 1.27 1.27)
+				)
+			)
+		)
+		(property "Mouser Part Number" "M20-7822046"
+			(at 123.19 76.2 0)
+			(hide yes)
+			(show_name no)
+			(do_not_autoplace no)
+			(effects
+				(font
+					(size 1.27 1.27)
+				)
+			)
+		)
+		(property "Manufacturer_Part_Number" "M20-7822046"
 			(at 123.19 76.2 0)
 			(hide yes)
@@
 			)
 		)
-		(property "Datasheet" ""
+		(property "Datasheet" "https://mm.digikey.com/Volume0/opasdata/d220001/medias/docus/937/Female_Headers.100_DS.pdf"
 			(at 137.16 76.2 0)
 			(hide yes)
@@
 		)
 		(property "Description" "Generic connector, single row, 01x20, script generated"
+			(at 137.16 76.2 0)
+			(hide yes)
+			(show_name no)
+			(do_not_autoplace no)
+			(effects
+				(font
+					(size 1.27 1.27)
+				)
+			)
+		)
+		(property "Mouser Part Number" "M20-7822046"
+			(at 137.16 76.2 0)
+			(hide yes)
+			(show_name no)
+			(do_not_autoplace no)
+			(effects
+				(font
+					(size 1.27 1.27)
+				)
+			)
+		)
+		(property "Manufacturer_Part_Number" "M20-7822046"
 			(at 137.16 76.2 0)
 			(hide yes)
@@
 			)
 		)
-		(property "Datasheet" ""
+		(property "Datasheet" "https://www.mouser.com/catalog/specsheets/YAGEO_PYu_RC_Group_51_RoHS_L_12.pdf"
 			(at 137.16 116.84 0)
 			(hide yes)
@@
 		(property "Description" "Resistor, US symbol"
 			(at 137.16 116.84 0)
+			(hide yes)
+			(show_name no)
+			(do_not_autoplace no)
+			(effects
+				(font
+					(size 1.27 1.27)
+				)
+			)
+		)
+		(property "Mouser Part Number" "RC0805FR-071KL"
+			(at 137.16 116.84 90)
+			(hide yes)
+			(show_name no)
+			(do_not_autoplace no)
+			(effects
+				(font
+					(size 1.27 1.27)
+				)
+			)
+		)
+		(property "Manufacturer_Part_Number" "RC0805FR-071KL"
+			(at 137.16 116.84 90)
 			(hide yes)
 			(show_name no)
@@
 			)
 		)
-		(property "Datasheet" ""
+		(property "Datasheet" "https://www.tme.eu/Document/a9f06aaefce48a31c93d25914fbf5b1b/B3F.PDF"
 			(at 125.73 111.76 0)
 			(hide yes)
@@
 			(at 125.73 116.84 0)
 			(hide yes)
+			(show_name no)
+			(do_not_autoplace no)
+			(effects
+				(font
+					(size 1.27 1.27)
+				)
+			)
+		)
+		(property "Mouser Part Number" "B3F-4000"
+			(at 125.73 116.84 0)
+			(hide yes)
+			(show_name no)
+			(do_not_autoplace no)
+			(effects
+				(font
+					(size 1.27 1.27)
+				)
+			)
+		)
+		(property "Manufacturer_Part_Number" "B3F-4000"
+			(at 125.73 116.84 0)
+			(hide yes)
