File: pcb/daughterboard/motors.kicad_sch (KiCad schematic)
At the start: 20 parts, among them J10 Conn_01x04_Socket, J11 Conn_01x04_Socket, J12 Conn_01x04_Socket, J13 Conn_01x04_Socket, J14 Conn_01x04_Socket, J15 Conn_01x04_Socket, J16 Conn_01x04_Socket, J17 Conn_01x04_Socket, J18 Conn_01x04_Socket, J19 Conn_01x04_Socket, J2 Conn_01x04_Socket, J20 Conn_01x04_Socket, J21 Conn_01x04_Socket, J3 Conn_01x04_Socket, J4 Conn_01x04_Socket, J5 Conn_01x04_Socket, J6 Conn_01x04_Socket, J7 Conn_01x04_Socket, J8 Conn_01x04_Socket, J9 Conn_01x04_Socket

Commit message: added footprints
Parts:
- J10, J11, J12, J13, J14, J15, J16, J17, J18, J19, J2, J20, J21, J3, J4, J5, J6, J7, J8, J9: footprint (none) -> A_HANU_FOOTPRINTS:52207-0633
Changed lines of the file:
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@@
 			)
 		)
-		(property "Footprint" ""
+		(property "Footprint" "A_HANU_FOOTPRINTS:52207-0633"
 			(at 143.51 92.71 0)
 			(hide yes)
@@
 			)
 		)
-		(property "Footprint" ""
+		(property "Footprint" "A_HANU_FOOTPRINTS:52207-0633"
 			(at 194.31 106.68 0)
 			(hide yes)
@@
 			)
 		)
-		(property "Footprint" ""
+		(property "Footprint" "A_HANU_FOOTPRINTS:52207-0633"
 			(at 40.64 29.21 0)
 			(hide yes)
@@
 			)
 		)
-		(property "Footprint" ""
+		(property "Footprint" "A_HANU_FOOTPRINTS:52207-0633"
 			(at 40.64 41.91 0)
 			(hide yes)
@@
 			)
 		)
-		(property "Footprint" ""
+		(property "Footprint" "A_HANU_FOOTPRINTS:52207-0633"
 			(at 91.44 55.88 0)
 			(hide yes)
@@
 			)
 		)
-		(property "Footprint" ""
+		(property "Footprint" "A_HANU_FOOTPRINTS:52207-0633"
 			(at 194.31 29.21 0)
 			(hide yes)
@@
 			)
 		)
-		(property "Footprint" ""
+		(property "Footprint" "A_HANU_FOOTPRINTS:52207-0633"
 			(at 91.44 29.21 0)
 			(hide yes)
@@
 			)
 		)
-		(property "Footprint" ""
+		(property "Footprint" "A_HANU_FOOTPRINTS:52207-0633"
 			(at 143.51 80.01 0)
 			(hide yes)
@@
 			)
 		)
-		(property "Footprint" ""
+		(property "Footprint" "A_HANU_FOOTPRINTS:52207-0633"
 			(at 92.71 92.71 0)
 			(hide yes)
@@
 			)
 		)
-		(property "Footprint" ""
+		(property "Footprint" "A_HANU_FOOTPRINTS:52207-0633"
 			(at 92.71 80.01 0)
 			(hide yes)
@@
 			)
 		)
-		(property "Footprint" ""
+		(property "Footprint" "A_HANU_FOOTPRINTS:52207-0633"
 			(at 142.24 29.21 0)
 			(hide yes)
@@
 			)
 		)
-		(property "Footprint" ""
+		(property "Footprint" "A_HANU_FOOTPRINTS:52207-0633"
 			(at 143.51 106.68 0)
 			(hide yes)
@@
 			)
 		)
-		(property "Footprint" ""
+		(property "Footprint" "A_HANU_FOOTPRINTS:52207-0633"
 			(at 40.64 55.88 0)
 			(hide yes)
@@
 			)
 		)
-		(property "Footprint" ""
+		(property "Footprint" "A_HANU_FOOTPRINTS:52207-0633"
 			(at 194.31 92.71 0)
 			(hide yes)
@@
 			)
 		)
-		(property "Footprint" ""
+		(property "Footprint" "A_HANU_FOOTPRINTS:52207-0633"
 			(at 194.31 80.01 0)
 			(hide yes)
@@
 			)
 		)
-		(property "Footprint" ""
+		(property "Footprint" "A_HANU_FOOTPRINTS:52207-0633"
 			(at 142.24 55.88 0)
 			(hide yes)
@@
 			)
 		)
-		(property "Footprint" ""
+		(property "Footprint" "A_HANU_FOOTPRINTS:52207-0633"
 			(at 194.31 55.88 0)
 			(hide yes)
@@
 			)
 		)
-		(property "Footprint" ""
+		(property "Footprint" "A_HANU_FOOTPRINTS:52207-0633"
 			(at 142.24 41.91 0)
 			(hide yes)
@@
 			)
 		)
-		(property "Footprint" ""
+		(property "Footprint" "A_HANU_FOOTPRINTS:52207-0633"
 			(at 194.31 41.91 0)
 			(hide yes)
@@
 			)
 		)
-		(property "Footprint" ""
+		(property "Footprint" "A_HANU_FOOTPRINTS:52207-0633"
 			(at 91.44 41.91 0)
 			(hide yes)
