File: pcb/daughterboard/drivers2.kicad_sch (KiCad schematic)
At the start: 12 parts, among them IC5 TLE94112ESXUMA1, IC6 TLE94112ESXUMA1, IC7 TLE94112ESXUMA1

Commit message: added footprints
Parts:
- C13, C14, C16, C17, C19, C20: footprint (none) -> A_HANU_FOOTPRINTS:CAPC0402X22N
- C15, C18, C21: footprint (none) -> A_HANU_FOOTPRINTS:CAPAE430X550N
- IC5, IC6, IC7: footprint SOP65P600X115-25N -> A_HANU_FOOTPRINTS:TLE94112ESXUMA1
Changed lines of the file:
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@@
 			)
 		)
-		(property "Footprint" ""
+		(property "Footprint" "A_HANU_FOOTPRINTS:CAPAE430X550N"
 			(at 247.65 106.68 0)
 			(hide yes)
@@
 			)
 		)
-		(property "Footprint" ""
+		(property "Footprint" "A_HANU_FOOTPRINTS:CAPAE430X550N"
 			(at 171.45 106.68 0)
 			(hide yes)
@@
 			)
 		)
-		(property "Footprint" ""
+		(property "Footprint" "A_HANU_FOOTPRINTS:CAPC0402X22N"
 			(at 242.57 106.68 0)
 			(hide yes)
@@
 			)
 		)
-		(property "Footprint" "SOP65P600X115-25N"
+		(property "Footprint" "A_HANU_FOOTPRINTS:TLE94112ESXUMA1"
 			(at 166.37 144.45 0)
 			(hide yes)
@@
 			)
 		)
-		(property "Footprint" ""
+		(property "Footprint" "A_HANU_FOOTPRINTS:CAPC0402X22N"
 			(at 63.5 105.41 0)
 			(hide yes)
@@
 			)
 		)
-		(property "Footprint" "SOP65P600X115-25N"
+		(property "Footprint" "A_HANU_FOOTPRINTS:TLE94112ESXUMA1"
 			(at 246.38 144.45 0)
 			(hide yes)
@@
 			)
 		)
-		(property "Footprint" ""
+		(property "Footprint" "A_HANU_FOOTPRINTS:CAPAE430X550N"
 			(at 87.63 106.68 0)
 			(hide yes)
@@
 			)
 		)
-		(property "Footprint" ""
+		(property "Footprint" "A_HANU_FOOTPRINTS:CAPC0402X22N"
 			(at 166.37 106.68 0)
 			(hide yes)
@@
 			)
 		)
-		(property "Footprint" ""
+		(property "Footprint" "A_HANU_FOOTPRINTS:CAPC0402X22N"
 			(at 223.52 105.41 0)
 			(hide yes)
@@
 			)
 		)
-		(property "Footprint" "SOP65P600X115-25N"
+		(property "Footprint" "A_HANU_FOOTPRINTS:TLE94112ESXUMA1"
 			(at 86.36 144.45 0)
 			(hide yes)
@@
 			)
 		)
-		(property "Footprint" ""
+		(property "Footprint" "A_HANU_FOOTPRINTS:CAPC0402X22N"
 			(at 82.55 106.68 0)
 			(hide yes)
@@
 			)
 		)
-		(property "Footprint" ""
+		(property "Footprint" "A_HANU_FOOTPRINTS:CAPC0402X22N"
 			(at 147.32 105.41 0)
 			(hide yes)

Commit message: initial design & routed decoupling capacitors
Parts:
- C15, C18, C21: footprint A_HANU_FOOTPRINTS:CAPAE430X550N -> A_HANU_FOOTPRINTS:T491A
Changed lines of the file:
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@@
 	(wire
 		(pts
+			(xy 25.4 110.49) (xy 36.83 110.49)
+		)
+		(stroke
+			(width 0)
+			(type default)
+		)
+	)
+	(wire
+		(pts
 			(xy 223.52 99.06) (xy 223.52 102.87)
 		)
@@
 	(wire
 		(pts
+			(xy 25.4 106.68) (xy 36.83 106.68)
+		)
+		(stroke
+			(width 0)
+			(type default)
+		)
+	)
+	(wire
+		(pts
 			(xy 168.91 101.6) (xy 166.37 101.6)
 		)
@@
 	)
 	(label "+3.3V"
+		(at 36.83 106.68 180)
+		(effects
+			(font
+				(size 1.27 1.27)
+				(thickness 0.254)
+				(bold yes)
+			)
+			(justify right bottom)
+		)
+	)
+	(label "+9V"
+		(at 36.83 110.49 180)
+		(effects
+			(font
+				(size 1 1)
+				(thickness 0.254)
+				(bold yes)
+			)
+			(justify right bottom)
+		)
+	)
+	(label "+3.3V"
 		(at 124.46 62.23 0)
 		(effects
@@
 			)
 		)
-		(property "Footprint" "A_HANU_FOOTPRINTS:CAPAE430X550N"
+		(property "Footprint" "A_HANU_FOOTPRINTS:T491A"
 			(at 247.65 106.68 0)
 			(hide yes)
@@
 			)
 		)
-		(property "Footprint" "A_HANU_FOOTPRINTS:CAPAE430X550N"
+		(property "Footprint" "A_HANU_FOOTPRINTS:T491A"
 			(at 171.45 106.68 0)
 			(hide yes)
@@
 	)
 	(symbol
+		(lib_id "power:+3.3V")
+		(at 25.4 106.68 90)
+		(unit 1)
+		(body_style 1)
+		(exclude_from_sim no)
+		(in_bom yes)
+		(on_board yes)
+		(in_pos_files yes)
+		(dnp no)
+		(fields_autoplaced yes)
+		(property "Reference" "#PWR028"
+			(at 29.21 106.68 0)
+			(hide yes)
+			(show_name no)
+			(do_not_autoplace no)
+			(effects
+				(font
+					(size 1.27 1.27)
+				)
+			)
+		)
+		(property "Value" "+3.3V"
+			(at 21.59 106.6799 90)
+			(show_name no)
+			(do_not_autoplace no)
+			(effects
+				(font
+					(size 1.27 1.27)
+				)
+				(justify left)
+			)
+		)
+		(property "Footprint" ""
+			(at 25.4 106.68 0)
+			(hide yes)
+			(show_name no)
+			(do_not_autoplace no)
+			(effects
+				(font
+					(size 1.27 1.27)
+				)
+			)
+		)
+		(property "Datasheet" ""
+			(at 25.4 106.68 0)
+			(hide yes)
+			(show_name no)
+			(do_not_autoplace no)
+			(effects
+				(font
+					(size 1.27 1.27)
+				)
+			)
+		)
+		(property "Description" "Power symbol creates a global label with name \"+3.3V\""
+			(at 25.4 106.68 0)
+			(hide yes)
+			(show_name no)
+			(do_not_autoplace no)
+			(effects
+				(font
+					(size 1.27 1.27)
+				)
+			)
+		)
+		(pin "1"
+		)
+		(instances
+			(project "daughterboard"
+				(path "/2255186e-2dec-4723-baeb-acb5f2843560/a102e0c2-7969-474b-a695-bbe14cacac49"
+					(reference "#PWR028")
+					(unit 1)
+				)
+			)
+		)
+	)
+	(symbol
 		(lib_id "Device:C_Small")
 		(at 242.57 106.68 0)
@@
 			)
 		)
-		(property "Footprint" "A_HANU_FOOTPRINTS:CAPAE430X550N"
+		(property "Footprint" "A_HANU_FOOTPRINTS:T491A"
 			(at 87.63 106.68 0)
 			(hide yes)
@@
 					(unit 1)
 				)
+			)
+		)
+	)
+	(symbol
+		(lib_id "power:+9V")
+		(at 25.4 110.49 90)
+		(unit 1)
+		(body_style 1)
+		(exclude_from_sim no)
+		(in_bom yes)
+		(on_board yes)
+		(in_pos_files yes)
+		(dnp no)
+		(fields_autoplaced yes)
+		(property "Reference" "#PWR029"
+			(at 29.21 110.49 0)
+			(hide yes)
+			(show_name no)
+			(do_not_autoplace no)
+			(effects
+				(font
+					(size 1.27 1.27)
+				)
+			)
+		)
+		(property "Value" "+9V"
+			(at 21.59 110.4899 90)
+			(show_name no)
+			(do_not_autoplace no)
+			(effects
+				(font
+					(size 1.27 1.27)
+				)
+				(justify left)
+			)
+		)
+		(property "Footprint" ""
+			(at 25.4 110.49 0)
+			(hide yes)
+			(show_name no)
+			(do_not_autoplace no)
+			(effects
+				(font
+					(size 1.27 1.27)
+				)
+			)
+		)
+		(property "Datasheet" ""
+			(at 25.4 110.49 0)
+			(hide yes)
+			(show_name no)
+			(do_not_autoplace no)
+			(effects
+				(font
+					(size 1.27 1.27)
+				)
+			)
+		)
+		(property "Description" "Power symbol creates a global label with name \"+9V\""
+			(at 25.4 110.49 0)
+			(hide yes)
+			(show_name no)
+			(do_not_autoplace no)
+			(effects
+				(font
+					(size 1.27 1.27)
+				)
+			)
+		)
+		(pin "1"
+		)
+		(instances
+			(project "daughterboard"
+				(path "/2255186e-2dec-4723-baeb-acb5f2843560/a102e0c2-7969-474b-a695-bbe14cacac49"
+					(reference "#PWR029")
+					(unit 1)
+				)
