File: pcb/motherboard/stm32.kicad_sch (KiCad schematic)
At the start: 18 parts, among them J1 BOOT PIN HEADER, J2 ST-Link, SW1 STM_RST, U1 STM32F103C8Tx, Y1 8MHz, Y2 32.768KHz

Commit message: added MCU hierarchy labels
Changed lines of the file:
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@@
 	)
 	(hierarchical_label "ADDR0"
-		(shape input)
+		(shape output)
 		(at 205.74 72.39 0)
 		(effects
@@
 	)
 	(hierarchical_label "SPI_CS"
-		(shape input)
+		(shape output)
 		(at 205.74 97.79 0)
 		(effects
@@
 	)
 	(hierarchical_label "ADDR1"
-		(shape input)
+		(shape output)
 		(at 205.74 74.93 0)
 		(effects
@@
 	)
 	(hierarchical_label "PB8"
-		(shape input)
+		(shape output)
 		(at 205.74 80.01 0)
 		(effects
@@
 	)
 	(hierarchical_label "SPI_MOSI"
-		(shape input)
+		(shape output)
 		(at 205.74 105.41 0)
 		(effects
@@
 	)
 	(hierarchical_label "UART_TX"
-		(shape input)
+		(shape output)
 		(at 205.74 107.95 0)
 		(effects
@@
 	)
 	(hierarchical_label "I2C_SDA"
-		(shape input)
+		(shape output)
 		(at 205.74 87.63 0)
 		(effects
@@
 	)
 	(hierarchical_label "ADDR2"
-		(shape input)
+		(shape output)
 		(at 205.74 77.47 0)
 		(effects
@@
 	)
 	(hierarchical_label "PB9"
-		(shape input)
+		(shape output)
 		(at 205.74 82.55 0)
 		(effects
@@
 	)
 	(hierarchical_label "SPI_CLK"
-		(shape input)
+		(shape output)
 		(at 205.74 100.33 0)
 		(effects
@@
 	)
 	(hierarchical_label "I2C_SCL"
-		(shape input)
+		(shape output)
 		(at 205.74 85.09 0)
 		(effects
